File: EPS/EPS.kicad_sch (KiCad schematic)
At the start: 37 parts, among them IC1 TPS63802DLAT, IC2 TPS63802DLAT, IC3 TPS63802DLAT, IC4 TPS63802DLAT, IC5 TPS63802DLAT, IC6 TPS63802DLAT

Commit message: Add files via upload
Al sistema EPS se le añadió el micro, y el componente encargado de la proteccion, hay que modificar las uniones todavia, y a ser posible añadir sensores para medir lo que nos interesa
Parts:
- removed IC2, IC3, IC5: TPS63802DLAT, TPS63802DLAT, symbol TPS63802DLAT:TPS63802DLAT
- added C1, C2, C3, C4: 0.1uF, Capacitor_SMD:C_0805_2012Metric, symbol Device:C
- added Cin1, Cin3, Cin4, Cin5, Cin6, Cin7, Cin8, Cin9, Cout7, Cout8, Cout9: 22uF, Capacitor_SMD:CP_Elec_6.3x4.5, symbol Device:C
- added Cin_EPS1, Cout_EPS1: 10uF, Capacitor_SMD:C_0805_2012Metric, symbol Device:C
- added D1, D2, D3, D4, D5, D6, D7, D8, D9: SS14, Diode_SMD:D_SMA, symbol Diode:SS14
- added H1, H2: Stack Header, Connector_PinHeader_2.54mm:PinHeader_2x26_P2.54mm_Vertical, symbol Connector_Generic:Conn_02x26_Odd_Even
- added IC10, IC12, IC14, IC16, IC18, IC8: TPS63802DLAT, SamacSys_Parts:TPS63802DLAT, symbol TPS63802DLAT:TPS63802DLAT
- added IC11, IC13, IC15, IC17, IC19, IC3, IC5, IC7, IC9: MP62551DJ-LF-Z, SOT95P280X100-6N, symbol MP62551DJ-LF-Z:MP62551DJ-LF-Z
- added IC2: STM32G474VET6, QFP50P1600X1600X160-100N, symbol STM32G474VET6:STM32G474VET6
- added L7, L8, L9: 470nH, Inductor_SMD:L_1206_3216Metric_Pad1.42x1.75mm_HandSolder, symbol Device:L
- added MH1, MH2, MH3, MH4: M3, MountingHole:MountingHole_3.2mm_M3_Pad, symbol Mechanical:MountingHole_Pad
- added Rfbb7, Rfbb8, Rfbb9: 91000, Resistor_SMD:R_0603_1608Metric, symbol Device:R
- added Rfbt7, Rfbt8, Rfbt9: 511000, Resistor_SMD:R_0603_1608Metric, symbol Device:R
- added Rpg7, Rpg8, Rpg9: 100000, Resistor_SMD:R_0603_1608Metric, symbol Device:R
- IC1, IC4, IC6: footprint TPS63802DLAT -> SamacSys_Parts:TPS63802DLAT
Connections:
- net +3.3V: now also Cout_EPS1.1, IC11.6 (OUT), IC13.6 (OUT), IC15.6 (OUT), IC17.6 (OUT), IC19.6 (OUT), IC3.6 (OUT), IC5.6 (OUT), IC7.6 (OUT), IC9.6 (OUT); no longer Cout1.1, Cout2.1, Cout3.1, Cout4.1, Cout5.1, Cout6.1, IC1.6 (VOUT), IC4.6 (VOUT), IC6.6 (VOUT), Rfbt1.1, Rfbt2.1, Rfbt3.1, Rfbt4.1, Rfbt5.1, Rfbt6.1, Rpg1.1, Rpg2.1, Rpg3.1, Rpg4.1, Rpg5.1, Rpg6.1
- net GND: now also C1.2, C2.2, C3.2, C4.2, Cin1.2, Cin3.2, Cin4.2, Cin5.2, Cin6.2, Cin7.2, Cin8.2, Cin9.2, Cin_EPS1.2, Cout7.2, Cout8.2, Cout9.2, Cout_EPS1.2, H2.21 (Pin_21), H2.22 (Pin_22), H2.29 (Pin_29), H2.30 (Pin_30), H2.31 (Pin_31), H2.32 (Pin_32), IC10.2 (MODE), IC10.3 (AGND), IC10.8 (GND), IC11.2 (GND), IC12.2 (MODE), IC12.3 (AGND), IC12.8 (GND), IC13.2 (GND), IC14.2 (MODE), IC14.3 (AGND), IC14.8 (GND), IC15.2 (GND), IC16.2 (MODE), IC16.3 (AGND), IC16.8 (GND), IC17.2 (GND), IC18.2 (MODE), IC18.3 (AGND), IC18.8 (GND), IC19.2 (GND), IC3.2 (GND), IC5.2 (GND), IC7.2 (GND), IC8.2 (MODE), IC8.3 (AGND), IC8.8 (GND), IC9.2 (GND), Rfbb7.2, Rfbb8.2, Rfbb9.2
- net at IC4.5 (PG): now also Rpg2.2; no longer Rpg4.2
- net at Rfbb6.1, Rfbt6.2: now also IC12.4 (FB); no longer IC6.4 (FB)
- net at IC6.5 (PG): now also Rpg3.2; no longer Rpg6.2
- net at L6.1: now also IC12.7 (L2); no longer IC6.7 (L2)
- net at L6.2: now also IC12.9 (L1); no longer IC6.9 (L1)
- net at Rfbb3.1, Rfbt3.2: now also IC6.4 (FB)
- net at L3.1: now also IC6.7 (L2)
- net at L3.2: now also IC6.9 (L1)
- net at Rfbb2.1, Rfbt2.2: now also IC4.4 (FB)
- net at Rfbb5.1, Rfbt5.2: now also IC10.4 (FB)
- net at Rfbb4.1, Rfbt4.2: now also IC8.4 (FB); no longer IC4.4 (FB)
- net at IC4.7 (L2): now also L2.1; no longer L4.1
- net at IC4.9 (L1): now also L2.2; no longer L4.2
- net at Rpg5.2: now also IC10.5 (PG)
- net at L5.1: now also IC10.7 (L2)
- net at L5.2: now also IC10.9 (L1)
- net Vin renamed Vin_EPS
- net Vin_EPS: now also Cin1.1, Cin3.1, Cin4.1, Cin5.1, Cin6.1, Cin7.1, Cin8.1, Cin9.1, Cin_EPS1.1, IC10.1 (EN), IC10.10 (VIN), IC12.1 (EN), IC12.10 (VIN), IC14.1 (EN), IC14.10 (VIN), IC16.1 (EN), IC16.10 (VIN), IC18.1 (EN), IC18.10 (VIN), IC8.1 (EN), IC8.10 (VIN)
- new net: C2.1, MH2.1
- new net: C4.1, MH4.1
- new net: C1.1, MH1.1
- new net: C3.1, MH3.1
- new net: Cout5.1, D5.2 (A), IC10.6 (VOUT), Rfbt5.1, Rpg5.1
- new net: Cout7.1, D7.2 (A), IC14.6 (VOUT), Rfbt7.1, Rpg7.1
- new net: Cout2.1, D1.2 (A), IC4.6 (VOUT), Rfbt2.1, Rpg2.1
- new net: IC18.4 (FB), Rfbb9.1, Rfbt9.2
- new net: IC18.5 (PG), Rpg9.2
- new net: Cout9.1, D9.2 (A), IC18.6 (VOUT), Rfbt9.1, Rpg9.1
- new net: IC18.7 (L2), L9.1
- new net: IC18.9 (L1), L9.2
- new net: Cout1.1, D2.2 (A), IC1.6 (VOUT), Rfbt1.1, Rpg1.1
- new net: Cout4.1, D4.2 (A), IC8.6 (VOUT), Rfbt4.1, Rpg4.1
- new net: D9.1 (K), IC19.1 (IN)
- new net: Cout3.1, D3.2 (A), IC6.6 (VOUT), Rfbt3.1, Rpg3.1
- new net: IC16.7 (L2), L8.1
- new net: IC16.9 (L1), L8.2
- new net: D6.1 (K), IC13.1 (IN)
- new net: Cout6.1, D6.2 (A), IC12.6 (VOUT), Rfbt6.1, Rpg6.1
- new net: IC16.4 (FB), Rfbb8.1, Rfbt8.2
- new net: IC16.5 (PG), Rpg8.2
- new net: Cout8.1, D8.2 (A), IC16.6 (VOUT), Rfbt8.1, Rpg8.1
- new net: IC14.5 (PG), Rpg7.2
- new net: IC12.5 (PG), Rpg6.2
- new net: IC8.5 (PG), Rpg4.2
- new net: D2.1 (K), IC3.1 (IN)
- new net: D3.1 (K), IC7.1 (IN)
- new net: IC14.7 (L2), L7.1
- new net: IC14.9 (L1), L7.2
- new net: D5.1 (K), IC11.1 (IN)
- new net: D7.1 (K), IC15.1 (IN)
- new net: D1.1 (K), IC5.1 (IN)
- new net: D4.1 (K), IC9.1 (IN)
- new net: IC8.7 (L2), L4.1
- new net: IC8.9 (L1), L4.2
- new net: IC14.4 (FB), Rfbb7.1, Rfbt7.2
- new net: D8.1 (K), IC17.1 (IN)
- new net +3V3: H2.27 (Pin_27), H2.28 (Pin_28)
- new net +5V: H2.25 (Pin_25), H2.26 (Pin_26)
- new net +BATT: H2.45 (Pin_45), H2.46 (Pin_46)
- new net 5VIN: H1.32 (Pin_32)
- new net BCR_OUT: H2.41 (Pin_41), H2.42 (Pin_42), H2.43 (Pin_43), H2.44 (Pin_44)
- new net CRX3/GP30: H1.29 (Pin_29)
- new net CS/GP10: H1.46 (Pin_46)
- new net CS/GP36: H1.50 (Pin_50)
- new net CS/GP37: H1.48 (Pin_48)
- new net CTX3/GP31: H1.31 (Pin_31)
- new net EN_0: IC2.20 (PA0), IC3.3 (EN)
- new net EN_1: IC2.21 (PA1), IC5.3 (EN)
- new net EN_2: IC2.22 (PA2), IC7.3 (EN)
- new net EN_3: IC2.25 (PA3), IC9.3 (EN)
- new net EN_4: IC11.3 (EN), IC2.26 (PA4)
- new net EN_5: IC13.3 (EN), IC2.27 (PA5)
- new net EN_6: IC15.3 (EN), IC2.28 (PA6)
- new net EN_7: IC17.3 (EN), IC2.29 (PA7)
- new net EN_8: IC19.3 (EN), IC2.69 (PA8)
- new net FLAG_0: IC2.32 (PB0), IC3.4 (~{FLAG})
- new net FLAG_1: IC2.33 (PB1), IC5.4 (~{FLAG})
- new net FLAG_2: IC2.34 (PB2), IC7.4 (~{FLAG})
- new net FLAG_3: IC2.90 (PB3), IC9.4 (~{FLAG})
- new net FLAG_4: IC11.4 (~{FLAG}), IC2.91 (PB4)
- new net FLAG_5: IC13.4 (~{FLAG}), IC2.92 (PB5)
- new net FLAG_6: IC15.4 (~{FLAG}), IC2.93 (PB6)
- new net FLAG_7: IC17.4 (~{FLAG}), IC2.94 (PB7)
- new net FLAG_8: IC19.4 (~{FLAG}), IC2.96 (PB9)
- new net GP14/A0/TX3: H1.15 (Pin_15)
- new net GP15/A1/RX3: H1.13 (Pin_13)
- new net GP2: H1.4 (Pin_4)
- new net GP20/A6/TX5: H1.19 (Pin_19)
- new net GP21/A7/RX5: H1.17 (Pin_17)
- new net GP22/A8: H1.18 (Pin_18)
- new net GP23/A9: H1.16 (Pin_16)
- new net GP3: H1.6 (Pin_6)
- new net GP32: H1.28 (Pin_28)
- new net GP33: H1.30 (Pin_30)
- new net GP38/A14: H1.26 (Pin_26)
- new net GP39/A15: H1.24 (Pin_24)
- new net GP4: H1.8 (Pin_8)
- new net GP40/A16: H1.22 (Pin_22)
- new net GP41/A17: H1.20 (Pin_20)
- new net GP5: H1.10 (Pin_10)
- new net GP6: H1.12 (Pin_12)
- new net GP9: H1.14 (Pin_14)
- new net MISO0: H1.38 (Pin_38)
- new net MISO1: H1.44 (Pin_44)
- new net MOSI0: H1.36 (Pin_36)
- new net MOSI1: H1.42 (Pin_42)
- new net PCM_IN: H2.35 (Pin_35), H2.36 (Pin_36)
- new net RX1/GP0: H1.5 (Pin_5)
- new net RX2/GP7: H1.9 (Pin_9)
- new net RX7/GP28: H1.21 (Pin_21)
- new net RX8/GP34: H1.25 (Pin_25)
- new net SCK0: H1.34 (Pin_34)
- new net SCK1: H1.40 (Pin_40)
- new net SCL0: H1.43 (Pin_43)
- new net SCL1: H1.39 (Pin_39)
- new net SCL2: H1.35 (Pin_35)
- new net SDA0: H1.41 (Pin_41)
- new net SDA1: H1.37 (Pin_37)
- new net SDA2: H1.33 (Pin_33)
- new net SW1: H2.9 (Pin_9)
- new net SW10: H2.18 (Pin_18)
- new net SW11: H2.19 (Pin_19)
- new net SW12: H2.20 (Pin_20)
- new net SW2: H2.10 (Pin_10)
- new net SW3: H2.11 (Pin_11)
- new net SW4: H2.12 (Pin_12)
- new net SW5: H2.13 (Pin_13)
- new net SW6: H2.14 (Pin_14)
- new net SW7: H2.15 (Pin_15)
- new net SW8: H2.16 (Pin_16)
- new net SW9: H2.17 (Pin_17)
- new net TX1/GP1: H1.7 (Pin_7)
- new net TX2/GP8: H1.11 (Pin_11)
- new net TX7/GP29: H1.23 (Pin_23)
- new net TX8/GP35: H1.27 (Pin_27)
- no-connect marks 0 -> 8
Other:
- title: EPS -> (none)
